File: hardware/mcu.kicad_sch (KiCad schematic)
At the start: 18 parts, among them J1 Conn_ARM_JTAG_SWD_10, SW1 B3U-1000P, SW2 B3U-1000P, U1 STM32G0B1KEUx

Commit message: add hardware revision v2
Parts:
- D3, D4: value GREEN -> YELLOW; footprint LED_SMD:LED_0402_1005Metric -> LED_SMD:LED_0603_1608Metric; Mfr. No 150040GS73220 -> 150060YS55040; Mouser No 710-150040GS73220 -> 710-150060YS55040
- D5, D6: value YELLOW -> GREEN; footprint LED_SMD:LED_0402_1005Metric -> LED_SMD:LED_0603_1608Metric; Mfr. No 150040YS73220 -> 150060GS55040; Mouser No 710-150040YS73220 -> 710-150060GS55040
- R3, R6: value 330Ω -> 100Ω; Mfr. Vishay -> YAGEO; Mfr. No CRCW0402330RJNEDC -> RC0402FR-07100RL; Mouser No 71-CRCW0402330RJNEDC -> 603-RC0402FR-07100RL
- R4, R5: value 330Ω -> 68Ω; Mfr. Vishay -> YAGEO; Mfr. No CRCW0402330RJNEDC -> RC0402FR-0768RL; Mouser No 71-CRCW0402330RJNEDC -> 603-RC0402FR-0768RL
Connections:
- net CAN1_ACT: now also U1.27 (PB3); no longer U1.26 (PA15)
- net CAN1_STA: now also U1.26 (PA15); no longer U1.27 (PB3)
- net at D5.1 (K): now also R3.1; no longer R5.1
- net at D3.1 (K): now also R5.1; no longer R3.1
Other:
- moved on the sheet: D3, D5
Changed lines of the file:
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@@
 	(title_block
 		(title "ubiquitous-waddle")
-		(date "2025-10-12")
-		(rev "v1")
+		(date "2025-12-22")
+		(rev "v2")
 		(company "leonwip <leonwip@proton.me>")
 		(comment 1 "CERN-OHL-P-2.0")
@@
 	)
 	(label "CAN1_ACT"
-		(at 142.24 106.68 0)
+		(at 86.36 91.44 180)
 		(effects
 			(font
 				(size 1.27 1.27)
 			)
-			(justify left bottom)
+			(justify right bottom)
 		)
 	)
@@
 	)
 	(label "CAN1_STA"
-		(at 86.36 91.44 180)
+		(at 142.24 106.68 0)
 		(effects
 			(font
 				(size 1.27 1.27)
 			)
-			(justify right bottom)
+			(justify left bottom)
 		)
 	)
@@
 	(symbol
 		(lib_id "Device:LED")
-		(at 215.9 58.42 90)
+		(at 241.3 58.42 90)
 		(unit 1)
 		(exclude_from_sim no)
@@
 		(fields_autoplaced yes)
 		(property "Reference" "D5"
-			(at 219.71 58.7374 90)
+			(at 245.11 58.7374 90)
 			(effects
 				(font
@@
 			)
 		)
-		(property "Value" "YELLOW"
-			(at 219.71 61.2774 90)
+		(property "Value" "GREEN"
+			(at 245.11 61.2774 90)
 			(effects
 				(font
@@
 			)
 		)
-		(property "Footprint" "LED_SMD:LED_0402_1005Metric"
-			(at 215.9 58.42 0)
+		(property "Footprint" "LED_SMD:LED_0603_1608Metric"
+			(at 241.3 58.42 0)
 			(effects
 				(font
@@
 		)
 		(property "Datasheet" "~"
-			(at 215.9 58.42 0)
+			(at 241.3 58.42 0)
 			(effects
 				(font
@@
 		)
 		(property "Description" "Light emitting diode"
-			(at 215.9 58.42 0)
+			(at 241.3 58.42 0)
 			(effects
 				(font
@@
 		)
 		(property "Sim.Pins" "1=K 2=A"
-			(at 215.9 58.42 0)
+			(at 241.3 58.42 0)
 			(effects
 				(font
@@
 			)
 		)
-		(property "Mouser No" "710-150040YS73220"
-			(at 215.9 58.42 90)
+		(property "Mouser No" "710-150060GS55040"
+			(at 241.3 58.42 90)
 			(effects
 				(font
@@
 			)
 		)
-		(property "Mfr. No" "150040YS73220"
-			(at 215.9 58.42 90)
+		(property "Mfr. No" "150060GS55040"
+			(at 241.3 58.42 90)
 			(effects
 				(font
@@
 		)
 		(property "Mfr." "Wurth Elektronik"
-			(at 215.9 58.42 90)
+			(at 241.3 58.42 90)
 			(effects
 				(font
@@
 			)
 		)
-		(property "Value" "YELLOW"
+		(property "Value" "GREEN"
 			(at 245.11 108.2674 90)
 			(effects
@@
 			)
 		)
-		(property "Footprint" "LED_SMD:LED_0402_1005Metric"
+		(property "Footprint" "LED_SMD:LED_0603_1608Metric"
 			(at 241.3 105.41 0)
 			(effects
@@
 			)
 		)
-		(property "Mouser No" "710-150040YS73220"
+		(property "Mouser No" "710-150060GS55040"
 			(at 241.3 105.41 90)
 			(effects
@@
 			)
 		)
-		(property "Mfr. No" "150040YS73220"
+		(property "Mfr. No" "150060GS55040"
 			(at 241.3 105.41 90)
 			(effects
@@
 			)
 		)
-		(property "Value" "330Ω"
+		(property "Value" "68Ω"
 			(at 218.44 69.8499 0)
 			(effects
@@
 			)
 		)
-		(property "Mouser No" "71-CRCW0402330RJNEDC"
+		(property "Mouser No" "603-RC0402FR-0768RL"
 			(at 215.9 68.58 0)
 			(effects
@@
 			)
 		)
-		(property "Mfr. No" "CRCW0402330RJNEDC"
+		(property "Mfr. No" "RC0402FR-0768RL"
 			(at 215.9 68.58 0)
 			(effects
@@
 			)
 		)
-		(property "Mfr." "Vishay"
+		(property "Mfr." "YAGEO"
 			(at 215.9 68.58 0)
 			(effects
@@
 			)
 		)
-		(property "Value" "330Ω"
+		(property "Value" "100Ω"
 			(at 243.84 116.8399 0)
 			(effects
@@
 			)
 		)
-		(property "Mouser No" "71-CRCW0402330RJNEDC"
+		(property "Mouser No" "603-RC0402FR-07100RL"
 			(at 241.3 115.57 0)
 			(effects
@@
 			)
 		)
-		(property "Mfr. No" "CRCW0402330RJNEDC"
+		(property "Mfr. No" "RC0402FR-07100RL"
 			(at 241.3 115.57 0)
 			(effects
@@
 			)
 		)
-		(property "Mfr." "Vishay"
+		(property "Mfr." "YAGEO"
 			(at 241.3 115.57 0)
 			(effects
@@
 	(symbol
 		(lib_id "Device:LED")
-		(at 241.3 58.42 90)
+		(at 215.9 58.42 90)
 		(unit 1)
 		(exclude_from_sim no)
@@
 		(fields_autoplaced yes)
 		(property "Reference" "D3"
-			(at 245.11 58.7374 90)
+			(at 219.71 58.7374 90)
 			(effects
 				(font
@@
 			)
 		)
-		(property "Value" "GREEN"
-			(at 245.11 61.2774 90)
+		(property "Value" "YELLOW"
+			(at 219.71 61.2774 90)
 			(effects
 				(font
@@
 			)
 		)
-		(property "Footprint" "LED_SMD:LED_0402_1005Metric"
-			(at 241.3 58.42 0)
+		(property "Footprint" "LED_SMD:LED_0603_1608Metric"
+			(at 215.9 58.42 0)
 			(effects
 				(font
@@
 		)
 		(property "Datasheet" "~"
-			(at 241.3 58.42 0)
+			(at 215.9 58.42 0)
 			(effects
 				(font
@@
 		)
 		(property "Description" "Light emitting diode"
-			(at 241.3 58.42 0)
+			(at 215.9 58.42 0)
 			(effects
 				(font
@@
 		)
 		(property "Sim.Pins" "1=K 2=A"
-			(at 241.3 58.42 0)
+			(at 215.9 58.42 0)
 			(effects
 				(font
@@
 			)
 		)
-		(property "Mouser No" "710-150040GS73220"
-			(at 241.3 58.42 90)
+		(property "Mouser No" "710-150060YS55040"
+			(at 215.9 58.42 90)
 			(effects
 				(font
@@
 			)
 		)
-		(property "Mfr. No" "150040GS73220"
-			(at 241.3 58.42 90)
+		(property "Mfr. No" "150060YS55040"
+			(at 215.9 58.42 90)
 			(effects
 				(font
@@
 		)
 		(property "Mfr." "Wurth Elektronik"
-			(at 241.3 58.42 90)
+			(at 215.9 58.42 90)
 			(effects
 				(font
@@
 			)
 		)
-		(property "Value" "330Ω"
+		(property "Value" "68Ω"
 			(at 218.44 116.8399 0)
 			(effects
@@
 			)
 		)
-		(property "Mouser No" "71-CRCW0402330RJNEDC"
+		(property "Mouser No" "603-RC0402FR-0768RL"
 			(at 215.9 115.57 0)
 			(effects
@@
 			)
 		)
-		(property "Mfr. No" "CRCW0402330RJNEDC"
+		(property "Mfr. No" "RC0402FR-0768RL"
 			(at 215.9 115.57 0)
 			(effects
@@
 			)
 		)
-		(property "Mfr." "Vishay"
+		(property "Mfr." "YAGEO"
 			(at 215.9 115.57 0)
 			(effects
@@
 			)
 		)
-		(property "Value" "330Ω"
+		(property "Value" "100Ω"
 			(at 243.84 69.8499 0)
 			(effects
@@
 			)
 		)
-		(property "Mouser No" "71-CRCW0402330RJNEDC"
+		(property "Mouser No" "603-RC0402FR-07100RL"
 			(at 241.3 68.58 0)
 			(effects
@@
 			)
 		)
-		(property "Mfr. No" "CRCW0402330RJNEDC"
+		(property "Mfr. No" "RC0402FR-07100RL"
 			(at 241.3 68.58 0)
 			(effects
@@
 			)
 		)
-		(property "Mfr." "Vishay"
+		(property "Mfr." "YAGEO"
 			(at 241.3 68.58 0)
 			(effects
@@
 			)
 		)
-		(property "Value" "GREEN"
+		(property "Value" "YELLOW"
 			(at 219.71 108.2674 90)
 			(effects
@@
 			)
 		)
-		(property "Footprint" "LED_SMD:LED_0402_1005Metric"
+		(property "Footprint" "LED_SMD:LED_0603_1608Metric"
 			(at 215.9 105.41 0)
 			(effects
@@
 			)
 		)
-		(property "Mouser No" "710-150040GS73220"
+		(property "Mouser No" "710-150060YS55040"
 			(at 215.9 105.41 90)
 			(effects
@@
 			)
 		)
-		(property "Mfr. No" "150040GS73220"
+		(property "Mfr. No" "150060YS55040"
 			(at 215.9 105.41 90)
 			(effects
