File: hardware/ubiquitous-waddle.kicad_pcb (KiCad board)
At the start: 4 copper layers, 56 x 32 mm, 44 parts, among them J1 Conn_ARM_JTAG_SWD_10, J2 DE9_Pins_MountingHoles, J3 USB_C_Receptacle_USB2.0_16P, SW1 B3U-1000P, SW2 B3U-1000P, U1 STM32G0B1KEUx, U2 MCP2542FDxMF, U3 MCP2542FDxMF, U4 824015043, U5 TLV75733PDRV

Commit message: add hardware revision v2
Parts:
- D3, D4: value GREEN -> YELLOW; footprint LED_SMD:LED_0402_1005Metric -> LED_SMD:LED_0603_1608Metric
- D5, D6: value YELLOW -> GREEN; footprint LED_SMD:LED_0402_1005Metric -> LED_SMD:LED_0603_1608Metric
- R3, R6: value 330Ω -> 100Ω
- R4, R5: value 330Ω -> 68Ω
- moved R3 1.20 mm to (142.0, 108.2)
- moved R5 1.20 mm to (140.8, 108.2)
- moved D4 0.50 mm to (147.1, 115.2)
- moved D6 0.50 mm to (150.5, 115.2)
- moved D3 0.50 mm to (140.3, 115.2)
- moved D5 0.50 mm to (143.7, 115.2)
- moved R10 0.10 mm to (125.0, 96.2)
- moved R9 0.10 mm to (123.9, 96.2)
Connections:
- R3 pad 1: Net-(D3-K) -> Net-(D5-K)
- R5 pad 1: Net-(D5-K) -> Net-(D3-K)
- U1 pad 26: /MCU/CAN1_ACT -> /MCU/CAN1_STA
- U1 pad 27: /MCU/CAN1_STA -> /MCU/CAN1_ACT
Other:
- board size 56 x 32 mm -> 53 x 32 mm
